Commit message: modified the 3d model, now it goes on the ground instead of into ground

File: urdf/my_robot_3d.urdf (robot description, URDF)
Before this commit: robot cartographer_backpack_3d, 4 links, 3 joints
Joints:
- joint imu_link_joint: origin xyz=0 0 0 rpy=3.1416 0 0 -> xyz=0 0 0 rpy=0 0 0
- joint laser_link_joint: origin xyz=0.19 0. 0.04 rpy=0. 1.3963 0. -> xyz=0.19 0. 0.04 rpy=0. 0. 0.
- joint toposens_link_joint: origin xyz=0.01 0. 0.19 rpy=0. -0.1745 3.1416 -> xyz=0.01 0. 0.19 rpy=0. 0. 0.

Commit message: changed the view in rviz, changed toposens position, continue on params adjusting

File: urdf/my_robot_3d.urdf (robot description, URDF)
Before this commit: robot cartographer_backpack_3d, 4 links, 3 joints
Joints:
- joint laser_link_joint: origin xyz=0.19 0. 0.04 rpy=0. 0. 0. -> xyz=0.01 0. 0.19 rpy=0. 0. 0.
- joint toposens_link_joint: origin xyz=0.01 0. 0.19 rpy=0. 0. 0. -> xyz=0.01 0. 0.7 rpy=0. 0. 0.
